Commit message: Fix ros2_control interfaces for bringup.

File: irb120pe_gazebo/urdf/irb120_ros2control.xacro (robot description, xacro)
@@ -208,16 +208,24 @@
       </xacro:unless>
       <!-- === SCHUNK EGP-64 GRIPPER === -->
-      <joint name="BASE_TF_joint">
-        <command_interface name="position"/>
-        <state_interface name="position"/>
-      </joint>
-      <joint name="TCP_joint">
-        <command_interface name="position"/>
-        <state_interface name="position"/>
-      </joint>
-      <joint name="EE_egp64_joint">
-        <command_interface name="position"/>
-        <state_interface name="position"/>
-      </joint>
+      <xacro:unless value="${bringup}">
+        <joint name="BASE_TF_joint">
+          <command_interface name="position"/>
+          <command_interface name="velocity"/>
+          <state_interface name="position"/>
+          <state_interface name="velocity"/>
+        </joint>
+        <joint name="TCP_joint">
+          <command_interface name="position"/>
+          <command_interface name="velocity"/>
+          <state_interface name="position"/>
+          <state_interface name="velocity"/>
+        </joint>
+        <joint name="EE_egp64_joint">
+          <command_interface name="position"/>
+          <command_interface name="velocity"/>
+          <state_interface name="position"/>
+          <state_interface name="velocity"/>
+        </joint>
+      </xacro:unless>
     </ros2_control>
     <xacro:unless value="${bringup}">
