Commit message: Modify limits in joint5 (safety).

File: irb120pe_gazebo/urdf/irb120_macro.urdf.xacro (robot description, xacro)
@@ -263,5 +263,5 @@
       <parent link="${prefix}link_4"/>
       <child link="${prefix}link_5"/>
-      <limit effort="1000" lower="-2.094395" upper="2.094395" velocity="5.58505"/>
+      <limit effort="1000" lower="-2.00" upper="2.00" velocity="5.58505"/> <!-- Joint5 limits lowered to +-2rad -->
       <axis xyz="0 1 0"/>
       <dynamics damping="2.0" friction="1.0"/>

File: irb120pe_gazebo/urdf/irb120_ros2control.xacro (robot description, xacro)
@@ -147,6 +147,6 @@
       <joint name="${prefix}joint_5">
         <command_interface name="position">
-          <param name="min">-2.094395</param>
-          <param name="max">2.094395</param>
+          <param name="min">-2.00</param>
+          <param name="max">2.00</param>  <!-- Joint5 limits lowered to +-2rad -->
         </command_interface>
         <command_interface name="velocity">

Commit message: Fix: Gripper (fixed) joints for bringup execution.

File: irb120pe_gazebo/urdf/irb120_macro.urdf.xacro (robot description, xacro)
@@ -438,12 +438,21 @@
       </collision>
     </link>
-    <joint name="egp64_finger_left_joint" type="prismatic" >
-      <parent link="egp64_gripper_base_link" />
-      <child link="egp64_finger_left_link" />
-      <limit effort="1000" lower="-0.001" upper="0.04" velocity="0.2"/>
-      <origin xyz="0.01483 -0.00782 0" rpy="0 0 0" />
-      <axis xyz="-1 0 0" />
-      <dynamics damping="1.0" friction="1.0"/>
-    </joint>
+    <xacro:unless value="${bringup}">
+      <joint name="egp64_finger_left_joint" type="prismatic" >
+        <parent link="egp64_gripper_base_link" />
+        <child link="egp64_finger_left_link" />
+        <limit effort="1000" lower="-0.001" upper="0.04" velocity="0.2"/>
+        <origin xyz="0.01483 -0.00782 0" rpy="0 0 0" />
+        <axis xyz="-1 0 0" />
+        <dynamics damping="1.0" friction="1.0"/>
+      </joint>
+    </xacro:unless>
+    <xacro:if value="${bringup}">
+      <joint name="egp64_finger_left_joint" type="fixed" >
+        <parent link="egp64_gripper_base_link" />
+        <child link="egp64_finger_left_link" />
+        <origin xyz="0.01483 -0.00782 0" rpy="0 0 0" />
+      </joint>
+    </xacro:if>
     <!-- LEFT FINGERTIP -->
     <link name="egp64_fingertip_left_link">
@@ -493,12 +502,21 @@
       </collision>
     </link>
-    <joint name="egp64_finger_right_joint" type="prismatic" >
-      <parent link="egp64_gripper_base_link" />
-      <child link="egp64_finger_right_link" />
-      <limit effort="1000" lower="-0.001" upper="0.04" velocity="0.2"/>
-      <origin xyz="-0.0153 -0.00602 0" rpy="0 0 0" />
-      <axis xyz="1 0 0" />
-      <dynamics damping="1.0" friction="1.0"/>
-    </joint>
+    <xacro:unless value="${bringup}">
+      <joint name="egp64_finger_right_joint" type="prismatic" >
+        <parent link="egp64_gripper_base_link" />
+        <child link="egp64_finger_right_link" />
+        <limit effort="1000" lower="-0.001" upper="0.04" velocity="0.2"/>
+        <origin xyz="-0.0153 -0.00602 0" rpy="0 0 0" />
+        <axis xyz="1 0 0" />
+        <dynamics damping="1.0" friction="1.0"/>
+      </joint>
+    </xacro:unless>
+    <xacro:if value="${bringup}">
+      <joint name="egp64_finger_right_joint" type="fixed" >
+        <parent link="egp64_gripper_base_link" />
+        <child link="egp64_finger_right_link" />
+        <origin xyz="-0.0153 -0.00602 0" rpy="0 0 0" />
+      </joint>
+    </xacro:if>
     <!-- RIGHT FINGERTIP -->
     <link name="egp64_fingertip_right_link">
