Commit message: Add camera to IRB120 enclosure.

File: irb120pe_gazebo/urdf/irb120.urdf.xacro (robot description, xacro)
@@ -111,3 +111,60 @@
     <origin xyz="-0.3 0.32 0.8605" rpy="0.0 0.0 0.0" />
   </joint>
+  <!-- CAMERA -->
+  <link name="camera_link">
+    <collision>
+      <origin xyz="0 0 0" rpy="0 0 0"/>
+      <geometry>
+        <box size="0.05 0.05 0.05"/>
+      </geometry>
+    </collision>
+    <visual>
+      <origin xyz="0 0 0" rpy="0 0 0"/>
+      <geometry>
+        <box size="0.05 0.05 0.05"/>
+      </geometry>
+    </visual>
+    <inertial>
+      <mass value="1.0" />
+      <origin xyz="0 0 0" rpy="0 0 0"/>
+      <inertia ixx="0.0" ixy="0.0" ixz="0.0" iyy="0.0" iyz="0.0" izz="0.0" />
+    </inertial>
+  </link>
+  <joint name="camera_joint" type="fixed">
+    <origin xyz="-0.15 0.65 1.90" rpy="0 1.23 3.1416"/>
+    <parent link="world"/>
+    <child link="camera_link"/>
+  </joint>
+  <gazebo reference="camera_link">
+    <sensor name="camera" type="camera">
+      <update_rate>30</update_rate>
+      <camera name="head">
+        <horizontal_fov>1.22</horizontal_fov>
+        <image>
+          <width>1920</width>
+          <height>1080</height>
+          <format>R8G8B8</format>
+        </image>
+        <clip>
+          <near>0.02</near>
+          <far>300</far>
+        </clip>
+        <noise>
+          <type>gaussian</type>
+          <mean>0.0</mean>
+          <stddev>0.007</stddev>
+        </noise>
+      </camera>
+      <plugin filename="libgazebo_ros_camera.so" name="camera_controller">
+        <robotNamespace/>
+        <alwaysOn>true</alwaysOn>
+        <updateRate>0.0</updateRate>
+        <cameraName>camera</cameraName>
+        <imageTopicName>image_raw</imageTopicName>
+        <cameraInfoTopicName>camera_info</cameraInfoTopicName>
+        <frameName>camera</frameName>
+        <hackBaseline>0.07</hackBaseline>
+      </plugin>
+    </sensor>
+  </gazebo>
 </robot>

Commit message: Add <unless bringup> tag for camera.

File: irb120pe_gazebo/urdf/irb120.urdf.xacro (robot description, xacro)
@@ -112,59 +112,61 @@
   </joint>
   <!-- CAMERA -->
-  <link name="camera_link">
-    <collision>
-      <origin xyz="0 0 0" rpy="0 0 0"/>
-      <geometry>
-        <box size="0.05 0.05 0.05"/>
-      </geometry>
-    </collision>
-    <visual>
-      <origin xyz="0 0 0" rpy="0 0 0"/>
-      <geometry>
-        <box size="0.05 0.05 0.05"/>
-      </geometry>
-    </visual>
-    <inertial>
-      <mass value="1.0" />
-      <origin xyz="0 0 0" rpy="0 0 0"/>
-      <inertia ixx="0.0" ixy="0.0" ixz="0.0" iyy="0.0" iyz="0.0" izz="0.0" />
-    </inertial>
-  </link>
-  <joint name="camera_joint" type="fixed">
-    <origin xyz="-0.15 0.65 1.90" rpy="0 1.23 3.1416"/>
-    <parent link="world"/>
-    <child link="camera_link"/>
-  </joint>
-  <gazebo reference="camera_link">
-    <sensor name="camera" type="camera">
-      <update_rate>30</update_rate>
-      <camera name="head">
-        <horizontal_fov>1.22</horizontal_fov>
-        <image>
-          <width>1920</width>
-          <height>1080</height>
-          <format>R8G8B8</format>
-        </image>
-        <clip>
-          <near>0.02</near>
-          <far>300</far>
-        </clip>
-        <noise>
-          <type>gaussian</type>
-          <mean>0.0</mean>
-          <stddev>0.007</stddev>
-        </noise>
-      </camera>
-      <plugin filename="libgazebo_ros_camera.so" name="camera_controller">
-        <robotNamespace/>
-        <alwaysOn>true</alwaysOn>
-        <updateRate>0.0</updateRate>
-        <cameraName>camera</cameraName>
-        <imageTopicName>image_raw</imageTopicName>
-        <cameraInfoTopicName>camera_info</cameraInfoTopicName>
-        <frameName>camera</frameName>
-        <hackBaseline>0.07</hackBaseline>
-      </plugin>
-    </sensor>
-  </gazebo>
+  <xacro:unless value="${bringup}">
+    <link name="camera_link">
+      <collision>
+        <origin xyz="0 0 0" rpy="0 0 0"/>
+        <geometry>
+          <box size="0.05 0.05 0.05"/>
+        </geometry>
+      </collision>
+      <visual>
+        <origin xyz="0 0 0" rpy="0 0 0"/>
+        <geometry>
+          <box size="0.05 0.05 0.05"/>
+        </geometry>
+      </visual>
+      <inertial>
+        <mass value="1.0" />
+        <origin xyz="0 0 0" rpy="0 0 0"/>
+        <inertia ixx="0.0" ixy="0.0" ixz="0.0" iyy="0.0" iyz="0.0" izz="0.0" />
+      </inertial>
+    </link>
+    <joint name="camera_joint" type="fixed">
+      <origin xyz="-0.15 0.65 1.90" rpy="0 1.23 3.1416"/>
+      <parent link="world"/>
+      <child link="camera_link"/>
+    </joint>
+    <gazebo reference="camera_link">
+      <sensor name="camera" type="camera">
+        <update_rate>30</update_rate>
+        <camera name="head">
+          <horizontal_fov>1.22</horizontal_fov>
+          <image>
+            <width>1920</width>
+            <height>1080</height>
+            <format>R8G8B8</format>
+          </image>
+          <clip>
+            <near>0.02</near>
+            <far>300</far>
+          </clip>
+          <noise>
+            <type>gaussian</type>
+            <mean>0.0</mean>
+            <stddev>0.007</stddev>
+          </noise>
+        </camera>
+        <plugin filename="libgazebo_ros_camera.so" name="camera_controller">
+          <robotNamespace/>
+          <alwaysOn>true</alwaysOn>
+          <updateRate>0.0</updateRate>
+          <cameraName>camera</cameraName>
+          <imageTopicName>image_raw</imageTopicName>
+          <cameraInfoTopicName>camera_info</cameraInfoTopicName>
+          <frameName>camera</frameName>
+          <hackBaseline>0.07</hackBaseline>
+        </plugin>
+      </sensor>
+    </gazebo>
+  </xacro:unless>
 </robot>

Commit message: Change coordinate frame origin and fix IRB120 urdf.

File: irb120pe_gazebo/urdf/irb120.urdf.xacro (robot description, xacro)
@@ -82,4 +82,5 @@
     <parent link="world"/>
     <child link="cell"/>
+    <origin xyz="0.926 -0.124 0.0" rpy="0.0 0.0 0.0" />
   </joint>
   <joint name="cell-base_link-fixed" type="fixed">

File: irb120pe_gazebo/urdf/irb120_macro.urdf.xacro (robot description, xacro)
@@ -520,11 +520,17 @@
     </link>
     <joint name="EE_egp64_joint" type="prismatic" >
-      <parent link="egp64_gripper_base_link" />
+      <parent link="tool0" />
       <child link="EE_egp64" />
       <limit effort="10000" lower="0.0" upper="0.0" velocity="0.0"/>
       <axis xyz="1 0 0" />
-      <origin xyz="0.033 -0.018 0.15" rpy="0 0 0"/>
+      <origin xyz="0.0 0.0 0.19" rpy="0 0 0"/>
     </joint>
     <!-- === SCHUNK EGP-64 GRIPPER === -->
+    <!-- LOAD LinkPose Gazebo (ROS2) PLUGIN: -->
+    <gazebo>
+      <plugin name="ros2_linkpose_plugin" filename="libros2_linkpose_plugin.so" >
+        <link>EE_egp64</link>
+      </plugin>
+    </gazebo>
   </xacro:macro>
 </robot>

File: irb120pe_gazebo/urdf/irb120_ros2control.xacro (robot description, xacro)
@@ -208,4 +208,16 @@
       </xacro:unless>
       <!-- === SCHUNK EGP-64 GRIPPER === -->
+      <joint name="BASE_TF_joint">
+        <command_interface name="position"/>
+        <state_interface name="position"/>
+      </joint>
+      <joint name="TCP_joint">
+        <command_interface name="position"/>
+        <state_interface name="position"/>
+      </joint>
+      <joint name="EE_egp64_joint">
+        <command_interface name="position"/>
+        <state_interface name="position"/>
+      </joint>
     </ros2_control>
     <xacro:unless value="${bringup}">

Commit message: Fix ros2_control warnings (bringup) and camera location.

File: irb120pe_gazebo/urdf/irb120.urdf.xacro (robot description, xacro)
@@ -134,5 +134,5 @@
     </link>
     <joint name="camera_joint" type="fixed">
-      <origin xyz="-0.15 0.65 1.90" rpy="0 1.23 3.1416"/>
+      <origin xyz="0.776 0.526 1.90" rpy="0 1.23 3.1416"/>
       <parent link="world"/>
       <child link="camera_link"/>

File: irb120pe_gazebo/urdf/irb120_macro.urdf.xacro (robot description, xacro)
@@ -311,11 +311,20 @@
       </visual>
     </link>
-    <joint name="BASE_TF_joint" type="prismatic" >
-      <parent link="base_link" />
-      <child link="BASE_TF" />
-      <limit effort="10000" lower="0.0" upper="0.0" velocity="0.0"/>
-      <axis xyz="1 0 0" />
-      <origin xyz="0.0 0.0 0.0" rpy="0 0 0"/>
-    </joint>
+    <xacro:unless value="${bringup}">
+      <joint name="BASE_TF_joint" type="prismatic" >
+        <parent link="base_link" />
+        <child link="BASE_TF" />
+        <limit effort="10000" lower="0.0" upper="0.0" velocity="0.0"/>
+        <axis xyz="1 0 0" />
+        <origin xyz="0.0 0.0 0.0" rpy="0 0 0"/>
+      </joint>
+    </xacro:unless>
+    <xacro:if value="${bringup}">
+      <joint name="BASE_TF_joint" type="fixed" >
+        <parent link="base_link" />
+        <child link="BASE_TF" />
+        <origin xyz="0.0 0.0 0.0" rpy="0 0 0"/>
+      </joint>
+    </xacro:if>
     <!-- EXTRA LINK + JOINT for the TCP to appear in Gazebo and to be able to calculate TRANSFORMS: -->
     <link name="TCP">
@@ -331,11 +340,20 @@
       </visual>
     </link>
-    <joint name="TCP_joint" type="prismatic" >
-      <parent link="${prefix}link_6" />
-      <child link="TCP" />
-      <limit effort="10000" lower="0.0" upper="0.0" velocity="0.0"/>
-      <axis xyz="1 0 0" />
-      <origin xyz="0.0 0.0 0.0" rpy="0 ${radians(90)} 0"/>
-    </joint>
+    <xacro:unless value="${bringup}">
+      <joint name="TCP_joint" type="prismatic" >
+        <parent link="${prefix}link_6" />
+        <child link="TCP" />
+        <limit effort="10000" lower="0.0" upper="0.0" velocity="0.0"/>
+        <axis xyz="1 0 0" />
+        <origin xyz="0.0 0.0 0.0" rpy="0 ${radians(90)} 0"/>
+      </joint>
+    </xacro:unless>
+    <xacro:if value="${bringup}">
+      <joint name="TCP_joint" type="fixed" >
+        <parent link="${prefix}link_6" />
+        <child link="TCP" />
+        <origin xyz="0.0 0.0 0.0" rpy="0 ${radians(90)} 0"/>
+      </joint>
+    </xacro:if>
     <!-- =================================== -->
     <!-- ========== END-EFFECTORS ========== -->
@@ -519,18 +537,27 @@
       </visual>
     </link>
-    <joint name="EE_egp64_joint" type="prismatic" >
-      <parent link="tool0" />
-      <child link="EE_egp64" />
-      <limit effort="10000" lower="0.0" upper="0.0" velocity="0.0"/>
-      <axis xyz="1 0 0" />
-      <origin xyz="0.0 0.0 0.19" rpy="0 0 0"/>
-    </joint>
+    <xacro:unless value="${bringup}">
+      <joint name="EE_egp64_joint" type="prismatic" >
+        <parent link="tool0" />
+        <child link="EE_egp64" />
+        <limit effort="10000" lower="0.0" upper="0.0" velocity="0.0"/>
+        <axis xyz="1 0 0" />
+        <origin xyz="0.0 0.0 0.19" rpy="0 0 0"/>
+      </joint>
+      <!-- LOAD LinkPose Gazebo (ROS2) PLUGIN: -->
+      <gazebo>
+        <plugin name="ros2_linkpose_plugin" filename="libros2_linkpose_plugin.so" >
+          <link>EE_egp64</link>
+        </plugin>
+      </gazebo>
+    </xacro:unless>
+    <xacro:if value="${bringup}">
+      <joint name="EE_egp64_joint" type="fixed" >
+        <parent link="tool0" />
+        <child link="EE_egp64" />
+        <origin xyz="0.0 0.0 0.19" rpy="0 0 0"/>
+      </joint>
+    </xacro:if>
     <!-- === SCHUNK EGP-64 GRIPPER === -->
-    <!-- LOAD LinkPose Gazebo (ROS2) PLUGIN: -->
-    <gazebo>
-      <plugin name="ros2_linkpose_plugin" filename="libros2_linkpose_plugin.so" >
-        <link>EE_egp64</link>
-      </plugin>
-    </gazebo>
   </xacro:macro>
 </robot>

Commit message: Add ArUco markers to Gazebo Simulation.

File: irb120pe_gazebo/urdf/irb120.urdf.xacro (robot description, xacro)
@@ -89,27 +89,99 @@
     <origin xyz="-0.6506 0.6489 0.8605" rpy="0.0 0.0 0.0" />
   </joint>
-  <link name="ergobox">
-    <visual>
-      <origin xyz="0.0 0.0 0.0" rpy="0 0 0" />
-      <geometry>
-        <mesh filename="file://$(find irb120pe_gazebo)/meshes/IALab/ergobox.dae" scale="1 1 1" />
-      </geometry>
-    </visual>
-    <collision>
-      <origin xyz="0.0 0.0 0.0" rpy="0 0 0" />
-      <geometry>
-        <mesh filename="file://$(find irb120pe_gazebo)/meshes/IALab/ergobox.dae" scale="1 1 1" />
-      </geometry>
-    </collision>
-    <inertial>
-      <mass value="10.0"/>
-      <inertia ixx="0.0002" ixy="0.0002" ixz="0.0002" iyy="0.0" iyz="0.0" izz="0.0" />
-    </inertial>
-  </link>
-  <joint name="cell-ergobox-fixed" type="fixed">
-    <parent link="cell"/>
-    <child link="ergobox"/>
-    <origin xyz="-0.3 0.32 0.8605" rpy="0.0 0.0 0.0" />
-  </joint>
+  <!-- ARUCO TAGS -->
+  <xacro:unless value="${bringup}">
+    <link name="aruco100">
+      <visual>
+        <origin xyz="0.0 0.0 0.0" rpy="0 0 0" />
+        <geometry>
+          <mesh filename="file://$(find irb120pe_gazebo)/meshes/aruco/aruco100.dae" scale="1 1 1" />
+        </geometry>
+      </visual>
+      <collision>
+        <origin xyz="0.0 0.0 0.0" rpy="0 0 0" />
+        <geometry>
+          <mesh filename="file://$(find irb120pe_gazebo)/meshes/aruco/aruco100.dae" scale="1 1 1" />
+        </geometry>
+      </collision>
+      <inertial>
+        <mass value="10.0"/>
+        <inertia ixx="0.0002" ixy="0.0002" ixz="0.0002" iyy="0.0" iyz="0.0" izz="0.0" />
+      </inertial>
+    </link>
+    <joint name="cell-aruco100-fixed" type="fixed">
+      <parent link="cell"/>
+      <child link="aruco100"/>
+      <origin xyz="-0.525 0.375 0.86" rpy="0.0 0.0 -1.5708" />
+    </joint>
+    <link name="aruco101">
+      <visual>
+        <origin xyz="0.0 0.0 0.0" rpy="0 0 0" />
+        <geometry>
+          <mesh filename="file://$(find irb120pe_gazebo)/meshes/aruco/aruco101.dae" scale="1 1 1" />
+        </geometry>
+      </visual>
+      <collision>
+        <origin xyz="0.0 0.0 0.0" rpy="0 0 0" />
+        <geometry>
+          <mesh filename="file://$(find irb120pe_gazebo)/meshes/aruco/aruco101.dae" scale="1 1 1" />
+        </geometry>
+      </collision>
+      <inertial>
+        <mass value="10.0"/>
+        <inertia ixx="0.0002" ixy="0.0002" ixz="0.0002" iyy="0.0" iyz="0.0" izz="0.0" />
+      </inertial>
+    </link>
+    <joint name="cell-aruco101-fixed" type="fixed">
+      <parent link="cell"/>
+      <child link="aruco101"/>
+      <origin xyz="-0.525 0.975 0.86" rpy="0.0 0.0 3.1416" />
+    </joint>
+    <link name="aruco102">
+      <visual>
+        <origin xyz="0.0 0.0 0.0" rpy="0 0 0" />
+        <geometry>
+          <mesh filename="file://$(find irb120pe_gazebo)/meshes/aruco/aruco102.dae" scale="1 1 1" />
+        </geometry>
+      </visual>
+      <collision>
+        <origin xyz="0.0 0.0 0.0" rpy="0 0 0" />
+        <geometry>
+          <mesh filename="file://$(find irb120pe_gazebo)/meshes/aruco/aruco102.dae" scale="1 1 1" />
+        </geometry>
+      </collision>
+      <inertial>
+        <mass value="10.0"/>
+        <inertia ixx="0.0002" ixy="0.0002" ixz="0.0002" iyy="0.0" iyz="0.0" izz="0.0" />
+      </inertial>
+    </link>
+    <joint name="cell-aruco102-fixed" type="fixed">
+      <parent link="cell"/>
+      <child link="aruco102"/>
+      <origin xyz="-0.225 0.375 0.86" rpy="0.0 0.0 0.0" />
+    </joint>
+    <link name="aruco103">
+      <visual>
+        <origin xyz="0.0 0.0 0.0" rpy="0 0 0" />
+        <geometry>
+          <mesh filename="file://$(find irb120pe_gazebo)/meshes/aruco/aruco103.dae" scale="1 1 1" />
+        </geometry>
+      </visual>
+      <collision>
+        <origin xyz="0.0 0.0 0.0" rpy="0 0 0" />
+        <geometry>
+          <mesh filename="file://$(find irb120pe_gazebo)/meshes/aruco/aruco103.dae" scale="1 1 1" />
+        </geometry>
+      </collision>
+      <inertial>
+        <mass value="10.0"/>
+        <inertia ixx="0.0002" ixy="0.0002" ixz="0.0002" iyy="0.0" iyz="0.0" izz="0.0" />
+      </inertial>
+    </link>
+    <joint name="cell-aruco103-fixed" type="fixed">
+      <parent link="cell"/>
+      <child link="aruco103"/>
+      <origin xyz="-0.225 0.975 0.86" rpy="0.0 0.0 1.5708" />
+    </joint>
+  </xacro:unless>
   <!-- CAMERA -->
   <xacro:unless value="${bringup}">

Commit message: Simplified Gz Simulation ready.

File: irb120pe_gazebo/urdf/irb120.urdf.xacro (robot description, xacro)
@@ -89,4 +89,28 @@
     <origin xyz="-0.6506 0.6489 0.8605" rpy="0.0 0.0 0.0" />
   </joint>
+  <!-- CubeTray -->
+  <link name="CubeTray">
+      <visual>
+        <origin xyz="0.0 0.0 0.0" rpy="0 0 0" />
+        <geometry>
+          <mesh filename="file://$(find irb120pe_gazebo)/meshes/IALab/irb120pe_CubeTray.dae" scale="1 1 1" />
+        </geometry>
+      </visual>
+      <collision>
+        <origin xyz="0.0 0.0 0.0" rpy="0 0 0" />
+        <geometry>
+          <mesh filename="file://$(find irb120pe_gazebo)/meshes/IALab/irb120pe_CubeTray.dae" scale="1 1 1" />
+        </geometry>
+      </collision>
+      <inertial>
+        <mass value="100.0"/>
+        <inertia ixx="0.0002" ixy="0.0002" ixz="0.0002" iyy="0.0" iyz="0.0" izz="0.0" />
+      </inertial>
+    </link>
+    <joint name="cell-CubeTray-fixed" type="fixed">
+      <parent link="cell"/>
+      <child link="CubeTray"/>
+      <origin xyz="-0.846 0.195 0.86" rpy="0.0 0.0 0.0" />
+    </joint>
   <!-- ARUCO TAGS -->
   <xacro:unless value="${bringup}">
@@ -112,5 +136,5 @@
       <parent link="cell"/>
       <child link="aruco100"/>
-      <origin xyz="-0.525 0.375 0.86" rpy="0.0 0.0 -1.5708" />
+      <origin xyz="-0.525 0.325 0.86" rpy="0.0 0.0 -1.5708" />
     </joint>
     <link name="aruco101">
@@ -158,5 +182,5 @@
       <parent link="cell"/>
       <child link="aruco102"/>
-      <origin xyz="-0.225 0.375 0.86" rpy="0.0 0.0 0.0" />
+      <origin xyz="-0.225 0.325 0.86" rpy="0.0 0.0 0.0" />
     </joint>
     <link name="aruco103">

Commit message: Add HMI_camera.

File: irb120pe_gazebo/urdf/irb120.urdf.xacro (robot description, xacro)
@@ -268,4 +268,61 @@
       </sensor>
     </gazebo>
+    <!-- CAMERA for R3M-HMI -->
+    <link name="HMI_camera_link">
+      <collision>
+        <origin xyz="0 0 0" rpy="0 0 0"/>
+        <geometry>
+          <box size="0.05 0.05 0.05"/>
+        </geometry>
+      </collision>
+      <visual>
+        <origin xyz="0 0 0" rpy="0 0 0"/>
+        <geometry>
+          <box size="0.05 0.05 0.05"/>
+        </geometry>
+      </visual>
+      <inertial>
+        <mass value="1.0" />
+        <origin xyz="0 0 0" rpy="0 0 0"/>
+        <inertia ixx="0.0" ixy="0.0" ixz="0.0" iyy="0.0" iyz="0.0" izz="0.0" />
+      </inertial>
+    </link>
+    <joint name="HMI_camera_joint" type="fixed">
+      <origin xyz="2.0 1.5 2.0" rpy="0 0.35 -2.6"/>
+      <parent link="world"/>
+      <child link="HMI_camera_link"/>
+    </joint>
+    <gazebo reference="HMI_camera_link">
+      <sensor name="HMI_camera" type="camera">
+        <update_rate>30</update_rate>
+        <camera name="head">
+          <horizontal_fov>1.22</horizontal_fov>
+          <image>
+            <width>1920</width>
+            <height>1080</height>
+            <format>R8G8B8</format>
+          </image>
+          <clip>
+            <near>0.02</near>
+            <far>300</far>
+          </clip>
+          <noise>
+            <type>gaussian</type>
+            <mean>0.0</mean>
+            <stddev>0.007</stddev>
+          </noise>
+        </camera>
+        <plugin filename="libgazebo_ros_camera.so" name="HMI_camera_controller">
+          <robotNamespace/>
+          <alwaysOn>true</alwaysOn>
+          <updateRate>0.0</updateRate>
+          <cameraName>HMI_camera</cameraName>
+          <imageTopicName>HMI_image_raw</imageTopicName>
+          <cameraInfoTopicName>HMI_camera_info</cameraInfoTopicName>
+          <frameName>HMI_camera</frameName>
+          <hackBaseline>0.07</hackBaseline>
+        </plugin>
+      </sensor>
+    </gazebo>
   </xacro:unless>
 </robot>
